File: CompVueloPotencia.kicad_sch (KiCad schematic)
At the start: 0 parts

Commit message: test for updates
Parts:
- added R1: R_Small, symbol Device:R_Small
- added U1: ESP32-S3-WROOM-1, RF_Module:ESP32-S3-WROOM-1, symbol RF_Module:ESP32-S3-WROOM-1
Connections:
- new net: U1.1 (GND), U1.40 (GND), U1.41 (GND)
Changed lines of the file:
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@@
 	(generator_version "9.0")
 	(paper "A4")
+	(symbol
+		(lib_id "Device:R_Small")
+		(at 74.93 64.77 0)
+		(unit 1)
+		(exclude_from_sim no)
+		(in_bom yes)
+		(on_board yes)
+		(dnp no)
+		(fields_autoplaced yes)
+		(property "Reference" "R1"
+			(at 77.47 63.4999 0)
+			(effects
+				(font
+					(size 1.016 1.016)
+				)
+				(justify left)
+			)
+		)
+		(property "Value" "R_Small"
+			(at 77.47 66.0399 0)
+			(effects
+				(font
+					(size 1.27 1.27)
+				)
+				(justify left)
+			)
+		)
+		(property "Footprint" ""
+			(at 74.93 64.77 0)
+			(effects
+				(font
+					(size 1.27 1.27)
+				)
+				(hide yes)
+			)
+		)
+		(property "Datasheet" "~"
+			(at 74.93 64.77 0)
+			(effects
+				(font
+					(size 1.27 1.27)
+				)
+				(hide yes)
+			)
+		)
+		(property "Description" "Resistor, small symbol"
+			(at 74.93 64.77 0)
+			(effects
+				(font
+					(size 1.27 1.27)
+				)
+				(hide yes)
+			)
+		)
+		(pin "1"
+		)
+		(pin "2"
+		)
+		(instances
+			(project ""
+				(path "/a84aba9c-0fb9-4754-89f4-1b118d6ea201"
+					(reference "R1")
+					(unit 1)
+				)
+			)
+		)
+	)
+	(symbol
+		(lib_id "RF_Module:ESP32-S3-WROOM-1")
+		(at 172.72 54.61 0)
+		(unit 1)
+		(exclude_from_sim no)
+		(in_bom yes)
+		(on_board yes)
+		(dnp no)
+		(fields_autoplaced yes)
+		(property "Reference" "U1"
+			(at 174.8633 24.13 0)
+			(effects
+				(font
+					(size 1.27 1.27)
+				)
+				(justify left)
+			)
+		)
+		(property "Value" "ESP32-S3-WROOM-1"
+			(at 174.8633 26.67 0)
+			(effects
+				(font
+					(size 1.27 1.27)
+				)
+				(justify left)
+			)
+		)
+		(property "Footprint" "RF_Module:ESP32-S3-WROOM-1"
+			(at 172.72 52.07 0)
+			(effects
+				(font
+					(size 1.27 1.27)
+				)
+				(hide yes)
+			)
+		)
+		(property "Datasheet" "https://www.espressif.com/sites/default/files/documentation/esp32-s3-wroom-1_wroom-1u_datasheet_en.pdf"
+			(at 172.72 54.61 0)
+			(effects
+				(font
+					(size 1.27 1.27)
+				)
+				(hide yes)
+			)
+		)
+		(property "Description" "RF Module, ESP32-S3 SoC, Wi-Fi 802.11b/g/n, Bluetooth, BLE, 32-bit, 3.3V, onboard antenna, SMD"
+			(at 172.72 54.61 0)
+			(effects
+				(font
+					(size 1.27 1.27)
+				)
+				(hide yes)
+			)
+		)
+		(pin "33"
+		)
+		(pin "34"
+		)
+		(pin "6"
+		)
+		(pin "8"
+		)
+		(pin "38"
+		)
+		(pin "7"
+		)
+		(pin "26"
+		)
+		(pin "14"
+		)
+		(pin "36"
+		)
+		(pin "3"
+		)
+		(pin "16"
+		)
+		(pin "30"
+		)
+		(pin "10"
+		)
+		(pin "32"
+		)
+		(pin "24"
+		)
+		(pin "12"
+		)
+		(pin "29"
+		)
+		(pin "40"
+		)
+		(pin "18"
+		)
+		(pin "17"
+		)
+		(pin "2"
+		)
+		(pin "28"
+		)
+		(pin "31"
+		)
+		(pin "21"
+		)
+		(pin "1"
+		)
+		(pin "20"
+		)
+		(pin "23"
+		)
+		(pin "19"
+		)
+		(pin "4"
+		)
+		(pin "13"
+		)
+		(pin "37"
+		)
+		(pin "11"
+		)
+		(pin "25"
+		)
+		(pin "15"
+		)
+		(pin "22"
+		)
+		(pin "41"
+		)
+		(pin "27"
+		)
+		(pin "9"
+		)
+		(pin "5"
+		)
+		(pin "35"
+		)
+		(pin "39"
+		)
+		(instances
+			(project ""
+				(path "/a84aba9c-0fb9-4754-89f4-1b118d6ea201"
+					(reference "U1")
+					(unit 1)
+				)
+			)
+		)
+	)
 	(sheet_instances
 		(path "/"
