File: CompVueloPotencia/3v3Outs.kicad_sch (KiCad schematic)
At the start: 4 parts

Commit message: Mcu Finishes, i think
Other:
- note added: "VIN: 6.5 V - 9 V VOUT: 3.3 V Iout_Max: 2A (ambas salidas)"
- note removed: "VIN: 6.5 V - 9 V VOUT: 3.3 V Iout_Max: 600 mA (Por salida)"
- company: (none) -> XIMBAL EK ELECTRONICA
Changed lines of the file:
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@@
 	(generator_version "9.99")
 	(paper "A5")
+	(title_block
+		(date "2025-09-10")
+		(rev "0.1")
+		(company "XIMBAL EK ELECTRONICA")
+	)
 	(rectangle
 		(start 67.31 50.8)
@@
 		)
 	)
-	(text "VIN: 		6.5 V - 9 V\nVOUT: 		3.3 V\nIout_Max: 	600 mA (Por salida)"
+	(text "VIN: 		6.5 V - 9 V\nVOUT: 		3.3 V\nIout_Max: 	2A (ambas salidas)"
 		(exclude_from_sim yes)
 		(at 20.32 21.844 0)
