File: CompVueloPotencia/BuckConv.kicad_sch (KiCad schematic)
At the start: 12 parts, among them U1 TPS5430DDA

Commit message: Mcu Finishes, i think
Parts:
- removed R4: 2k2, Resistor_SMD:R_0805_2012Metric, symbol Device:R_Small
- removed R5: 10k, Resistor_SMD:R_0805_2012Metric, symbol Device:R_Small
- R3: value 2k2 -> 3k
Connections:
- net GND: now also R3.2
Other:
- note added: "VIN: 6.6 V - 9 V VOUT: 5.3 V Iout_Max: 3 A"
- note removed: "BUCK CONVERTER WITH TPS5430"
- note removed: "R_Equivalente: aprox 3.05k"
- note removed: "VIN: 6.5 V - 9 V VOUT: 5.2 V Iout_Max: 3 A"
- company: (none) -> XIMBAL EK ELECTRONICA
- moved on the sheet: R3
