File: CompVueloPotencia/BuckConv3v3.kicad_sch (KiCad schematic)
At the start: 11 parts, among them U2 TPS5430DDA

Commit message: Mcu Finishes, i think
Other:
- company: (none) -> XIMBAL EK ELECTRONICA
Changed lines of the file:
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@@
 	(generator_version "9.99")
 	(paper "A5")
+	(title_block
+		(date "2025-09-10")
+		(rev "0.1")
+		(company "XIMBAL EK ELECTRONICA")
+	)
 	(rectangle
 		(start 120.65 57.15)
