File: CompVueloPotencia/CompVueloPotencia.kicad_pcb (KiCad board)
At the start: 2 copper layers, 58 parts, among them J1 Conn_01x02, SW1 Reset, SW2 SW_SPDT_312, SW3 SW_SPDT_312, U1 TPS5430DDA, U2 TPS5430DDA, U3 STM32F103CBT6, U4 LD39200DPUR, U5 LD39200DPUR

Commit message: Mcu Finishes, i think
Parts:
- removed R5: 10k, Resistor_SMD:R_0805_2012Metric
- removed SW2: SW_SPDT_312, Button_Switch_THT:SW_Slide-03_Wuerth-WS-SLTV_10x2.5x6.4_P2.54mm
- added C26: 9pF, Resistor_SMD:R_0805_2012Metric, F.Cu at (182.4, 59.5)
- added J2: USB_B_Micro, Connector_USB:USB_Micro-B_Amphenol_10118194_Horizontal, F.Cu at (189.6, 58.2)
- added J3: ST_LINK, Connector_PinHeader_2.54mm:PinHeader_1x04_P2.54mm_Vertical, F.Cu at (177.9, 57.4)
- added SW4: SW_SPDT, SPDT_Big:SolderWire-0.5sqmm_1x03_P4.8mm_D0.9mm_OD2.3mm, F.Cu at (178.6, 51.0)
- added Y1: 16MHz, Crystal:Crystal_SMD_3225-4Pin_3.2x2.5mm, F.Cu at (191.3, 70.0)
- C11, C17: value 10u -> 10uF
- C12, C14, C15, C16: value 100n -> 100nF
- C13: value 100n -> 9pF; footprint Capacitor_SMD:C_0805_2012Metric -> Resistor_SMD:R_0805_2012Metric
- C18, C19: value 1u -> 1uF
- R1: value 10K -> 1k5
- R3: value 2k2 -> 3k
- R4: value 2k2 -> 10k
- moved C1 56.6 mm to (109.0, 48.5)
- moved R4 45.9 mm to (182.4, 65.4)
- moved C13 40.5 mm to (182.4, 56.6)
- moved SW1 29.6 mm to (87.7, 36.1)
- moved R1 19.4 mm to (182.4, 62.5)
Connections:
- C1 pad 1: ESP32_EN -> NRST
- C11 pad 1: VDD -> 3V3_MCU
- C12 pad 1: VDD -> 3V3_MCU
- C13 pad 1: NRST -> OSC_OUT
- C14 pad 1: VDD -> 3V3_MCU
- C15 pad 1: VDD -> 3V3_MCU
- C16 pad 1: VDD -> 3V3_MCU
- C19 pad 1: VDD -> 3V3_MCU
- FB1 pad 2: VDD -> 3V3_MCU
- R1 pad 1: +3.3V -> 3V3_MCU
- R1 pad 2: ESP32_EN -> USB_D+
- R3 pad 2: Net-(R3-Pad2) -> GND
- R4 pad 1: Net-(R3-Pad2) -> Net-(SW4-B)
- R4 pad 2: GND -> BOOT0
- SW1 pad 2: ESP32_EN -> NRST
- U3 pad 1: VDD -> 3V3_MCU
- U3 pad 10: unconnected-(U3-PA0-Pad10) -> /MCU/ADC_IN0
- U3 pad 11: unconnected-(U3-PA1-Pad11) -> /MCU/ADC_IN1
- U3 pad 12: unconnected-(U3-PA2-Pad12) -> /MCU/ADC_IN2
- U3 pad 13: unconnected-(U3-PA3-Pad13) -> /MCU/ADC_IN3
- U3 pad 14: unconnected-(U3-PA4-Pad14) -> /MCU/CS
- U3 pad 15: unconnected-(U3-PA5-Pad15) -> /MCU/SCLK
- U3 pad 16: unconnected-(U3-PA6-Pad16) -> /MCU/MISO
- U3 pad 17: unconnected-(U3-PA7-Pad17) -> /MCU/MOSI
- U3 pad 18: unconnected-(U3-PB0-Pad18) -> /MCU/ADC_IN8
- U3 pad 19: unconnected-(U3-PB1-Pad19) -> /MCU/ADC_IN9
- U3 pad 21: unconnected-(U3-PB10-Pad21) -> /MCU/UART3_TX
- U3 pad 22: unconnected-(U3-PB11-Pad22) -> /MCU/UART3_RX
- U3 pad 23: Net-(U3-VSS-Pad23) -> GND
- U3 pad 24: VDD -> 3V3_MCU
- U3 pad 32: unconnected-(U3-PA11-Pad32) -> USB_D-
- U3 pad 33: unconnected-(U3-PA12-Pad33) -> USB_D+
- U3 pad 34: unconnected-(U3-PA13-Pad34) -> SWDIO
- U3 pad 35: Net-(U3-VSS-Pad23) -> GND
- U3 pad 36: VDD -> 3V3_MCU
- U3 pad 37: unconnected-(U3-PA14-Pad37) -> SWCLK
- U3 pad 42: unconnected-(U3-PB6-Pad42) -> /MCU/SCL
- U3 pad 43: unconnected-(U3-PB7-Pad43) -> /MCU/SDA
- U3 pad 44: unconnected-(U3-BOOT0-Pad44) -> BOOT0
- U3 pad 47: Net-(U3-VSS-Pad23) -> GND
- U3 pad 48: VDD -> 3V3_MCU
- U3 pad 5: unconnected-(U3-PD0-Pad5) -> OSC_IN
- U3 pad 6: unconnected-(U3-PD1-Pad6) -> OSC_OUT
- U3 pad 8: unconnected-(U3-VSSA-Pad8) -> GND

Commit message: little changes
Parts:
- SW3: footprint Connector_Wire:SolderWire-0.5sqmm_1x03_P4.8mm_D0.9mm_OD2.3mm -> SPDT_Big:SolderWire-0.5sqmm_1x03_P4.8mm_D0.9mm_OD2.3mm
- moved U1 11.6 mm to (87.3, 67.2)
Changed lines of the file:
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@@
 		)
 		(embedded_fonts no)
+		(model "C:/Users/vickh/Documents/KiCadPrj/PCBCompVuelo-PotenciaKicad/Footprints/LD39200DPUR_3D/LD39200DPUR.step"
+			(offset
+				(xyz 0 0 0)
+			)
+			(scale
+				(xyz 1 1 1)
+			)
+			(rotate
+				(xyz -90 -0 -0)
+			)
+		)
 	)
 	(footprint "Capacitor_SMD:C_0805_2012Metric"
@@
 		)
 		(embedded_fonts no)
+		(model "C:/Users/vickh/Documents/KiCadPrj/PCBCompVuelo-PotenciaKicad/Footprints/LD39200DPUR_3D/LD39200DPUR.step"
+			(offset
+				(xyz 0 0 0)
+			)
+			(scale
+				(xyz 1 1 1)
+			)
+			(rotate
+				(xyz -90 -0 -0)
+			)
+		)
 	)
 	(footprint "Capacitor_SMD:C_0805_2012Metric"
@@
 		)
 	)
-	(footprint "Connector_Wire:SolderWire-0.5sqmm_1x03_P4.8mm_D0.9mm_OD2.3mm"
+	(footprint "SPDT_Big:SolderWire-0.5sqmm_1x03_P4.8mm_D0.9mm_OD2.3mm"
 		(layer "F.Cu")
 		(at 63.6 53.93)
@@
 		(tags "connector wire 0.5sqmm")
 		(property "Reference" "SW3"
-			(at 4.8 -2.35 0)
+			(at 5.2 -3 0)
 			(layer "F.SilkS")
 			(effects
@@
 		)
 		(property "Value" "SW_SPDT_312"
-			(at 4.8 2.35 0)
+			(at 4.8 3 0)
 			(layer "F.Fab")
 			(effects
@@
 		(duplicate_pad_numbers_are_jumpers no)
 		(fp_line
+			(start -2.1 1.5)
+			(end -2.1 -1.5)
+			(stroke
+				(width 0.1)
+				(type default)
+			)
+			(layer "F.SilkS")
+		)
+		(fp_line
+			(start -1.7 -1.9)
+			(end 11.4 -1.9)
+			(stroke
+				(width 0.1)
+				(type default)
+			)
+			(layer "F.SilkS")
+		)
+		(fp_line
+			(start 11.487868 1.8)
+			(end -1.8 1.8)
+			(stroke
+				(width 0.1)
+				(type default)
+			)
+			(layer "F.SilkS")
+		)
+		(fp_line
+			(start 11.8 -1.5)
+			(end 11.8 1.5)
+			(stroke
+				(width 0.1)
+				(type default)
+			)
+			(layer "F.SilkS")
+		)
+		(fp_arc
+			(start -2.1 -1.5)
+			(mid -1.982843 -1.782843)
+			(end -1.7 -1.9)
+			(stroke
+				(width 0.1)
+				(type default)
+			)
+			(layer "F.SilkS")
+		)
+		(fp_arc
+			(start -1.8 1.8)
+			(mid -2.012132 1.712132)
+			(end -2.1 1.5)
+			(stroke
+				(width 0.1)
+				(type default)
+			)
+			(layer "F.SilkS")
+		)
+		(fp_arc
+			(start 11.4 -1.9)
+			(mid 11.682843 -1.782843)
+			(end 11.8 -1.5)
+			(stroke
+				(width 0.1)
+				(type default)
+			)
+			(layer "F.SilkS")
+		)
+		(fp_arc
+			(start 11.787868 1.5)
+			(mid 11.7 1.712132)
+			(end 11.487868 1.8)
+			(stroke
+				(width 0.1)
+				(type default)
+			)
+			(layer "F.SilkS")
+		)
+		(fp_line
 			(start -1.9 -1.65)
 			(end -1.9 1.65)
@@
 	(footprint "Package_SO:TI_SO-PowerPAD-8_ThermalVias"
 		(layer "F.Cu")
-		(at 78.8 75.095)
+		(at 87.35 67.225)
 		(descr "8-pin HTSOP package with 1.27mm pin pitch, compatible with SOIC-8, 3.9x4.9mm² body, exposed pad, thermal vias with large copper area, as proposed in http://www.ti.com/lit/ds/symlink/tps5430.pdf")
 		(tags "HTSOP 1.27")
