File: CompVueloPotencia/CompVueloPotencia.kicad_sch (KiCad schematic)
At the start: 3 parts, among them J1 Conn_01x02, SW2 SW_SPDT_312, SW3 SW_SPDT_312

Commit message: Mcu Finishes, i think
Parts:
- removed SW2: SW_SPDT_312, Button_Switch_THT:SW_Slide-03_Wuerth-WS-SLTV_10x2.5x6.4_P2.54mm, symbol Switch:SW_SPDT_312
Other:
- sheet MCU ports: added ADC_IN0, ADC_IN1, ADC_IN2, ADC_IN3, ADC_IN8, ADC_IN9, CS, UART3_RX, UART3_TX; removed CS0, CS1
- note removed: "Prog/Enable"
- company: (none) -> XIMBAL EK ELECTRONICA
- moved on the sheet: J1, SW3

Commit message: little changes
Parts:
- SW3: footprint Connector_Wire:SolderWire-0.5sqmm_1x03_P4.8mm_D0.9mm_OD2.3mm -> SPDT_Big:SolderWire-0.5sqmm_1x03_P4.8mm_D0.9mm_OD2.3mm
Changed lines of the file:
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@@
 			)
 		)
-		(property "Footprint" "Connector_Wire:SolderWire-0.5sqmm_1x03_P4.8mm_D0.9mm_OD2.3mm"
+		(property "Footprint" "SPDT_Big:SolderWire-0.5sqmm_1x03_P4.8mm_D0.9mm_OD2.3mm"
 			(at 29.21 69.85 0)
 			(hide yes)
