File: CompVueloPotencia/McuStm32.kicad_sch (KiCad schematic)
At the start: 13 parts, among them SW1 Reset, U3 STM32F103CBT6

Commit message: Mcu Finishes, i think
Parts:
- added C13, C26: 9pF, Resistor_SMD:R_0805_2012Metric, symbol Device:C_Small
- added J2: USB_B_Micro, Connector_USB:USB_Micro-B_Amphenol_10118194_Horizontal, symbol Connector:USB_B_Micro
- added J3: ST_LINK, Connector_PinHeader_2.54mm:PinHeader_1x04_P2.54mm_Vertical, symbol Connector_Generic:Conn_01x04
- added R4: 10k, Resistor_SMD:R_0805_2012Metric, symbol Device:R_Small
- added SW4: SW_SPDT, SPDT_Big:SolderWire-0.5sqmm_1x03_P4.8mm_D0.9mm_OD2.3mm, symbol Switch:SW_SPDT_312
- added Y1: 16MHz, Crystal:Crystal_SMD_3225-4Pin_3.2x2.5mm, symbol Device:Crystal_GND24
- R1: value 10K -> 1k5
Connections:
- net GND: now also U3.23 (VSS), U3.35 (VSS), U3.47 (VSS), U3.8 (VSSA), C13.2, C26.2, J2.5 (GND), J2.6 (Shield), J3.4 (Pin_4), SW4.3 (A), Y1.2, Y1.4
- net MISO: now also U3.16 (PA6)
- net MOSI: now also U3.17 (PA7)
- net NRST: no longer R1.2
- net SCL: now also U3.42 (PB6)
- net SCLK: now also U3.15 (PA5)
- net SDA: now also U3.43 (PB7)
- net VDD: now also J3.1 (Pin_1), SW4.2 (C)
- net ADC_IN0: now reaches U3.10 (PA0)
- net ADC_IN1: now reaches U3.11 (PA1)
- net ADC_IN2: now reaches U3.12 (PA2)
- net ADC_IN3: now reaches U3.13 (PA3)
- net CS: now reaches U3.14 (PA4)
- net ADC_IN8: now reaches U3.18 (PB0)
- net ADC_IN9: now reaches U3.19 (PB1)
- net UART3_TX: now reaches U3.21 (PB10)
- net UART3_RX: now reaches U3.22 (PB11)
- net USB_D-: now reaches U3.32 (PA11)
- net USB_D-: now also J2.2 (D-)
- net USB_D+: now reaches U3.33 (PA12)
- net USB_D+: now also R1.2, J2.3 (D+)
- net SWDIO: now reaches U3.34 (PA13)
- net SWDIO: now also J3.2 (Pin_2)
- net SWCLK: now reaches U3.37 (PA14)
- net SWCLK: now also J3.3 (Pin_3)
- net BOOT0: now reaches U3.44 (BOOT0)
- net BOOT0: now also R4.2
- net OSC_IN: now reaches U3.5 (PD0)
- net OSC_IN: now also C26.1, Y1.1
- net OSC_OUT: now reaches U3.6 (PD1)
- net OSC_OUT: now also C13.1, Y1.3
- new net: R4.1, SW4.1 (B)
- new net VBUS: J2.1 (VBUS)
- no-connect marks 0 -> 1
Other:
- note added: "CRYSTAL osc"
- note added: "DECOUPLING CAP."
- note added: "Microcontroller Unit (MCU)"
- note added: "RESET & BOOT selector"
- note added: "USB & STLINK Connector"
- note added: "VDDA Filtering"
- company: (none) -> XIMBAL EK ELECTRONICA
- title: (none) -> STM32F103CBT6  Integration Schematic
- moved on the sheet: C1, C11, C12, C14, C15, C16, C17, C18, C19, FB1, SW1, U3
