File: SupplyBoard/PCB/5VBuckReg.kicad_sch (KiCad schematic)
At the start: 10 parts, among them U8 TPS5430DDA

Commit message: Supply Board & Folder Organization
Reorganization of the power supply board components, simplifying the layout to facilitate future debugging and reorganizing some folders and documents, as well as adding the power supply board schematic; in supply board only need to make the routing
Parts:
- D3: footprint Diode_SMD:D_SMA-SMB_Universal_Handsoldering -> Diode_SMD:D_SMA
Changed lines of the file:
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@@
 			)
 		)
-		(property "Footprint" "Diode_SMD:D_SMA-SMB_Universal_Handsoldering"
+		(property "Footprint" "Diode_SMD:D_SMA"
 			(at 116.84 43.18 90)
 			(effects
