File: SupplyBoard/PCB/Reg_Sense.kicad_sch (KiCad schematic)
At the start: 5 parts, among them J4 Conn_01x03

Commit message: Supply & Coms-Sensor Board
la organizacion de los componentes presentes en las placas, se quedaran de esa manera, se espera que en la serigrafia se incluyan los logos de los patrocinadores, ademas se incluyo la carpeta 3D la cual contiene modelos en 3D de las dos placas, con serigrafia y componentes incluidos y ya
Parts:
- J4: footprint Connector_PinHeader_2.54mm:PinHeader_1x03_P2.54mm_Vertical -> Connector_JST:JST_XH_S3B-XH-A_1x03_P2.50mm_Horizontal
Changed lines of the file:
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@@
 			)
 		)
-		(property "Footprint" "Connector_PinHeader_2.54mm:PinHeader_1x03_P2.54mm_Vertical"
+		(property "Footprint" "Connector_JST:JST_XH_S3B-XH-A_1x03_P2.50mm_Horizontal"
 			(at 35.56 82.55 0)
 			(effects
