File: CompVuelo_V2.0/mcustm32.kicad_sch (KiCad schematic)
At the start: 1 part, among them U1 STM32F446RETx

Commit message: prueba0
mostrar avance
Parts:
- added C1, C2, C3, C4, C7, C8, C9: 100nF, symbol Device:C_Small
- added C10, C11: 20pf, symbol Device:C_Small
- added C5, C6: 10uF, symbol Device:C_Small
- added FB1: 120R, symbol Device:FerriteBead_Small
- added R1: 10k, symbol Device:R_Small
- added SW1: SW_Push, symbol Switch:SW_Push
- added SW2: SW_SPDT, symbol Switch:SW_SPDT
- added Y1: 26Mhz, Crystal:Crystal_SMD_SeikoEpson_TSX3225-4Pin_3.2x2.5mm, symbol Device:Crystal_GND23_Small
Connections:
- net +3V3: now reaches U1.1 (VBAT)
- net +3V3: now also U1.19 (VDD), U1.32 (VDD), U1.48 (VDD), U1.64 (VDD), C1.1, C2.1, C3.1, C4.1, C5.1, C8.1, FB1.1, SW2.3 (C)
- net GND: now reaches U1.12 (VSSA)
- net GND: now also U1.18 (VSS), U1.31 (VSS), U1.47 (VSS), U1.63 (VSS), C1.2, C10.2, C11.2, C2.2, C3.2, C4.2, C5.2, C6.2, C7.2, C8.2, C9.2, SW1.1, SW2.1 (A), Y1.2, Y1.3
- net VDDA: now reaches U1.13 (VDDA)
- net VDDA: now also C6.1, C7.1, FB1.2
- net RECU_{1}: now reaches U1.26 (PB0)
- net RECU_{2}: now reaches U1.27 (PB1)
- net SWDIO: now reaches U1.46 (PA13)
- net SWCLK: now reaches U1.49 (PA14)
- net OSC_IN: now reaches U1.5 (PH0)
- net OSC_IN: now also C11.1, Y1.1
- net SPI_{SCK}: now reaches U1.55 (PB3)
- net UART_{1}_TX: now reaches U1.58 (PB6)
- net UART_{1}_RX: now reaches U1.59 (PB7)
- net OSC_OUT: now reaches U1.6 (PH1)
- net OSC_OUT: now also C10.1, Y1.4
- net BOOT0: now reaches U1.60 (BOOT0)
- net BOOT0: now also R1.2
- net SCL: now reaches U1.61 (PB8)
- net SDA: now reaches U1.62 (PB9)
- net NRST: now reaches U1.7 (NRST)
- net NRST: now also C9.1, SW1.2
- new net: R1.1, SW2.2 (B)
Other:
- moved on the sheet: U1
